File: TPS5430Buck/TPS5430Buck.kicad_sch (KiCad schematic)
At the start: 15 parts, among them J11 Screw_Terminal_01x02, J12 Conn_01x03_Pin, U3 TPS5430DDA

Commit message: TPS5430Buck: fuse re-annotation (F10->F8, F9->F7) and project settings rewritten by newer KiCad
Uncommitted state carried over from the former TPS5430Buck repo.

Co-Authored-By: Claude Opus 5.5 <noreply@anthropic.com>
Parts:
- renumbered F9 to F7, F10 to F8
Changed lines of the file:
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@@
 		(dnp no)
 		(fields_autoplaced yes)
-		(property "Reference" "F10"
+		(property "Reference" "F8"
 			(at 227.33 63.5 90)
 			(show_name no)
@@
 			(project "TPS5430Buck"
 				(path "/abc0b92f-ec94-4587-a0dc-b6ae56d461f6"
-					(reference "F10")
+					(reference "F8")
 					(unit 1)
 				)
@@
 		(dnp no)
 		(fields_autoplaced yes)
-		(property "Reference" "F9"
+		(property "Reference" "F7"
 			(at 102.87 63.5 90)
 			(show_name no)
@@
 			(project "TPS5430Buck"
 				(path "/abc0b92f-ec94-4587-a0dc-b6ae56d461f6"
-					(reference "F9")
-					(unit 1)
-				)
+					(reference "F7")
+					(unit 1)
+				)
